File: Tests/test-data/example-sch.sch (EAGLE design)
At the start: 20 parts, among them J1 DIP16SOCKET, J2 DIP16SOCKET, U10 74LS174N, U11 74LS174N, U12 74ALS27N, U13 74LS174N, U14 74180N, U17 74LS123N, U18 SN15836N, U2 HD6821P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

Commit message: Symbols and DeviceSets are now loaded
Parts:
- added U1: LM555_DIP, IC_Clock-Timing:LM555_DIP
- added U16: 74180N, 74ttl-din:74180N
- R3: device Resistor:R-US_AXIAL-7.2MM-PITCH -> Resistor:R-US_AXIAL-11.7MM-PITCH
Other:
- moved on the sheet: U9A, U9B, U9C
